File: Hardware/electric-imp-shield.brd (EAGLE design)
At the start: 59.7 x 53.3 mm, 37 parts, among them Q2 BSS138, Q3 BSS138, U1 ELECTRIC_IMP, U2 ARDUINO_SHIELD, U3 MIC5219-3.3, U4 ATSHA204-TSU

Commit message: Updating to new socket fp, 0603 packages, schematic updates
Parts:
- added FRAME1: FRAME-LETTER, SparkFun-Retired:CREATIVE_COMMONS
- added U$6: REVISION, SparkFun-Aesthetics:REVISION
- C1, C4: device SparkFun-Passives:0402-CAP -> SparkFun-Capacitors:0603-CAP
- C3, C5: device SparkFun-Passives:EIA3216 -> SparkFun-Capacitors:EIA3216
- R1, R10, R2, R3, R6, R7, R8, R9: device SparkFun-Passives:0402-RES -> SparkFun-Resistors:0603-RES
- U1: device SparkFun-RF:SD_MMC_SOCKET -> SparkFun-RF:SD_1:1
- moved U1 29.2 mm to (30.5, 24.1), turned to 0 degrees
- moved C1 2.54 mm to (24.1, 27.9), turned to 180 degrees
Connections:
- net GND: now also U1.SH@1, U1.SH@2; no longer U1.S1, U1.S2
Routing:
- net GND: track 2.59 -> 0.00 mm
- net PIN7: track 46.2 -> 48.7 mm
- net PIN5: track 50.9 -> 53.3 mm
- net CD: track 32.8 -> 35.0 mm
- net PIN9: track 44.4 -> 45.3 mm
- net N$2: track 6.24 -> 6.88 mm
Other:
- board text added: "Jim Lindblom"
- board text added: "Toni Klopfenstein"
